File: Alcantara_v.1.0.sch (KiCad schematic (older format))
At the start: 22 parts, among them IC3 TLV803EA30DCKR, J5 PJS008U-3000-0, J8 53261-0527, Q1 MMSS8050-H-TP, Q2 MMSS8050-H-TP

Commit message: Add files via upload
Parts:
- IC3: symbol SamacSys_Parts:TLV803EA30DCKR -> Alcantara_v.1.0-rescue:TLV803EA30DCKR-SamacSys_Parts
- J5: symbol SamacSys_Parts:PJS008U-3000-0 -> Alcantara_v.1.0-rescue:PJS008U-3000-0-SamacSys_Parts
- J8: symbol SamacSys_Parts:53261-0527 -> Alcantara_v.1.0-rescue:53261-0527-SamacSys_Parts
- MOD1: symbol dk_RF-Transceiver-Modules:ESP32-WROOM-32 -> Alcantara_v.1.0-rescue:ESP32-WROOM-32-dk_RF-Transceiver-Modules
- Q1, Q2: symbol dk_Transistors-Bipolar-BJT-Single:MMSS8050-H-TP -> Alcantara_v.1.0-rescue:MMSS8050-H-TP-dk_Transistors-Bipolar-BJT-Single
- S4, S5: symbol SamacSys_Parts:EVP-AAM02W -> Alcantara_v.1.0-rescue:EVP-AAM02W-SamacSys_Parts
Other:
- note removed: "> 4 camadas go BRRRRRRRR"
- note removed: "> Conferir o pinout dos botões de EN e IO0"
- note removed: "> Editar silk dos botões"
- note removed: "> Escolher uma chave deslizante para o liga/desliga"
- note removed: "> Mover o capacitor e resistor de reset mais pra perto\n da ESP"
- note removed: "> Mudar o conector micro USB para um 100% SMD"
- note removed: "> Ou ligar junto ao RGB principal"
- note removed: "> Ponderar sobre a possibilidade de retirar os LEDs do FTDI"
- note removed: ">Refletir sobre quais decisões me trouxeram até aqui"
- note removed: "LISTA DE AFAZERES"
Changed lines of the file:
@@
 encoding utf-8
 Sheet 1 4
-Title "Alcantara V.1.0"
-Date "2021-06-08"
-Rev ""
+Title "Alcântara "
+Date "2021-10-05"
+Rev "1.0"
 Comp "Zenith Aerospace"
 Comment1 ""
@@
 	9750 5650 9850 5650
 $Comp
-L dk_RF-Transceiver-Modules:ESP32-WROOM-32 MOD1
+L Alcantara_v.1.0-rescue:ESP32-WROOM-32-dk_RF-Transceiver-Modules MOD1
 U 1 1 60CDB9CF
 P 4550 5150
@@
 	9750 5000 9850 5000
 $Comp
-L dk_Transistors-Bipolar-BJT-Single:MMSS8050-H-TP Q1
+L Alcantara_v.1.0-rescue:MMSS8050-H-TP-dk_Transistors-Bipolar-BJT-Single Q1
 U 1 1 61214E60
 P 8350 3900
@@
 $EndComp
 $Comp
-L dk_Transistors-Bipolar-BJT-Single:MMSS8050-H-TP Q2
+L Alcantara_v.1.0-rescue:MMSS8050-H-TP-dk_Transistors-Bipolar-BJT-Single Q2
 U 1 1 61215ACB
 P 8350 4500
@@
 Verificar que os pinos conectados em VP e VN não flutuarão, \nse não um pullup será necessário nesses pinos. Ele não possui\npullup interno.
 $Comp
-L SamacSys_Parts:EVP-AAM02W S5
+L Alcantara_v.1.0-rescue:EVP-AAM02W-SamacSys_Parts S5
 U 1 1 60E2AB97
 P 4950 3350
@@
 	6200 3450 6200 3650
 $Comp
-L SamacSys_Parts:EVP-AAM02W S4
+L Alcantara_v.1.0-rescue:EVP-AAM02W-SamacSys_Parts S4
 U 1 1 60E6112B
 P 1950 3500
@@
 Wire Wire Line
 	3200 3600 3200 3800
-Wire Notes Line
-	14700 0    14700 8250
-Wire Notes Line
-	14700 8250 11850 8250
-Wire Notes Line
-	11850 8250 11850 0
-Wire Notes Line
-	11850 0    14700 0
-Text Notes 12700 250  0    79   Italic 16
-LISTA DE AFAZERES
-Text Notes 12150 600  0    50   ~ 0
-> Mudar o conector micro USB para um 100% SMD
-Text Notes 12150 750  0    50   ~ 0
-> Escolher uma chave deslizante para o liga/desliga
-Text Notes 12150 900  0    50   ~ 0
-> Conferir o pinout dos botões de EN e IO0
-Text Notes 12150 1050 0    50   ~ 0
-> Editar silk dos botões
-Text Notes 12150 1200 0    50   ~ 0
-> Ponderar sobre a possibilidade de retirar os LEDs do FTDI
-Text Notes 12150 1550 0    50   ~ 0
->Refletir sobre quais decisões me trouxeram até aqui
-Text Notes 12250 1350 0    50   ~ 0
-> Ou ligar junto ao RGB principal
 Text GLabel 4000 5750 0    50   Input ~ 0
 GPS_TIMEPULSE
@@
 Wire Wire Line
 	7850 6200 7700 6200
-Text Notes 12150 1950 0    50   ~ 0
-> Mover o capacitor e resistor de reset mais pra perto\n   da ESP
-Text Notes 12150 1700 0    50   ~ 0
-> 4 camadas go BRRRRRRRR
 Wire Wire Line
 	3400 3250 3750 3250
@@
 $EndComp
 $Comp
-L SamacSys_Parts:PJS008U-3000-0 J5
+L Alcantara_v.1.0-rescue:PJS008U-3000-0-SamacSys_Parts J5
 U 1 1 612F4333
 P 3000 1650
@@
 $EndComp
 $Comp
-L SamacSys_Parts:53261-0527 J8
+L Alcantara_v.1.0-rescue:53261-0527-SamacSys_Parts J8
 U 1 1 61489378
 P 7750 5050
@@
 	7300 5950 7300 6050
 $Comp
-L SamacSys_Parts:TLV803EA30DCKR IC3
+L Alcantara_v.1.0-rescue:TLV803EA30DCKR-SamacSys_Parts IC3
 U 1 1 612F7BFE
 P 2150 3300
