File: Telecommunications.sch (KiCad schematic (older format))
At the start: 15 parts, among them J1 U_FL-R-SMT_10_, J2 142-0701-801, J3 142-0701-801, U1 E22-900M30S, U4 NEO-M8N

Commit message: Add files via upload
Parts:
- J2, J3: symbol dk_Coaxial-Connectors-RF:142-0701-801 -> Alcantara_v.1.0-rescue:142-0701-801-dk_Coaxial-Connectors-RF
- U1: symbol E22_Radios_Zenith:E22-900M30S -> Alcantara_v.1.0-rescue:E22-900M30S-E22_Radios_Zenith
Changed lines of the file:
@@
 NoConn ~ 3900 4450
 $Comp
-L dk_Coaxial-Connectors-RF:142-0701-801 J2
+L Alcantara_v.1.0-rescue:142-0701-801-dk_Coaxial-Connectors-RF J2
 U 1 1 60E543A4
 P 5300 4950
@@
 	9400 4300 9450 4300
 $Comp
-L dk_Coaxial-Connectors-RF:142-0701-801 J?
+L Alcantara_v.1.0-rescue:142-0701-801-dk_Coaxial-Connectors-RF J?
 U 1 1 60FC2F34
 P 10500 3850
@@
 Connection ~ 7500 4800
 $Comp
-L E22_Radios_Zenith:E22-900M30S U1
+L Alcantara_v.1.0-rescue:E22-900M30S-E22_Radios_Zenith U1
 U 1 1 612EA8AF
 P 8850 4350
