File: Alcantara_v.1.0.kicad_pcb (KiCad board)
At the start: 4 copper layers, 105.4 x 36.8 mm, 85 parts, among them IC1 TLV809ED29DBZR, IC2 MAX17201G+T, IC3 TLV803EA30DCKR, J1 U_FL-R-SMT_10_, J2 142-0701-801, J3 142-0701-801, J4 USB_B_Micro, J5 PJS008U-3000-0, J8 53261-0527, Q1 MMSS8050-H-TP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

Commit message: Updated RF section ground planes.
Parts:
- removed the G*** at (120.6, 32.0)
- removed the G*** at (122.6, 41.8)
- added G***: LOGO, LogosZenith:AlcantaraLogoReto_1,8mm, B.Cu at (128.1, 32.1)
- added G***: LOGO, LogosZenith:Logo_10,8mm, B.Cu at (101.6, 32.1)
- added Q7: 2N7002NXAKR, SamacSys_Parts:SOT95P230X110-3N, B.Cu at (112.8, 55.9)
- added R29: 10, Resistor_SMD:R_0603_1608Metric, F.Cu at (112.4, 63.6)
- added R33: 330, Resistor_SMD:R_0603_1608Metric, B.Cu at (117.3, 55.9)
- added R34: 10K, Resistor_SMD:R_0603_1608Metric, B.Cu at (115.6, 55.9)
- added S6: MSS-102545-14A-V-SMT, Downloaded:SW_MSS-102545-14A-V-SMT, B.Cu at (116.8, 62.9)
- C10: footprint Capacitor_SMD:CP_Elec_5x3 -> Capacitor_SMD:CP_Elec_5x5.3
- R8: value 10K -> 10; moved to F.Cu
- moved R8 7.76 mm to (120.5, 63.4)
- moved R22 7.72 mm to (117.7, 55.7)
- moved R6 7.45 mm to (119.0, 55.9)
- moved D2 6.77 mm to (113.2, 59.9), turned to 0 degrees
- moved R21 6.55 mm to (115.1, 55.7)
- moved R20 4.57 mm to (112.4, 55.7)
- moved R23 2.92 mm to (120.5, 55.6)
- moved C15 0.50 mm to (100.7, 56.7)
- moved L2 0.34 mm to (97.2, 56.7)
- moved C14 0.06 mm to (109.1, 35.0)
Connections:
- C15 pad 2: GND -> GNDA
- IC1 pad 1: /Power Management/Pack -> Net-(IC1-Pad1)
- J1 pad 2: GND -> GNDA
- J2 pad 2: GND -> GNDA
- MOD1 pad 14: GPS_TIMEPULSE -> GPS_ON_OFF
- R6 pad 2: GPS_TIMEPULSE -> GPS_ON_OFF
- R8 pad 1: GPS_TIMEPULSE -> Net-(R29-Pad2)
- R8 pad 2: GND -> /Power Management/Pack
- U2 pad 11: Net-(IC1-Pad3) -> Net-(IC1-Pad1)
- U4 pad 10: GND -> GNDA
- U4 pad 12: GND -> GNDA
- U4 pad 13: GND -> GND1
- U4 pad 24: GND -> GND1
- U4 pad 3: GPS_TIMEPULSE -> Net-(U4-Pad3)
- U4 pad 7: GND -> GND1
Routing:
- net GPS_TIMEPULSE: track 46.4 -> 0.00 mm, vias 4 -> 0
- net GND1: track 0.00 -> 46.3 mm, vias 0 -> 3
- net Net-(IC1-Pad3): track 3.75 -> 50.0 mm, vias 0 -> 2
- net /Power Management/Pack: track 106.9 -> 153.0 mm, vias 0 -> 2
- net GPS_ON_OFF: track 0.00 -> 23.1 mm, vias 0 -> 2
- net GND: track 88.1 -> 71.3 mm, vias 144 -> 133
- net Net-(R29-Pad2): track 0.00 -> 15.2 mm, vias 0 -> 1
- net Net-(J3-Pad2): track 15.8 -> 5.21 mm, vias 0 -> 12
- net +3V3: track 109.2 -> 100.6 mm, vias 15 -> 16
- net RGB_LED_B: track 18.1 -> 25.9 mm
- net RGB_LED_G: track 21.2 -> 14.3 mm
- net Net-(J1-Pad1): track 21.8 -> 27.8 mm
- net GNDA: track 0.00 -> 4.51 mm, vias 0 -> 28
- net Net-(Q7-Pad1): track 0.00 -> 3.40 mm
- net Net-(IC1-Pad1): track 0.00 -> 2.66 mm
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- added copper zone on B.Cu, net GNDA
- added copper zone on In2.Cu, net GNDA
- added copper zone on B.Cu, net Net-(J3-Pad2)
- added copper zone on In2.Cu, net Net-(J3-Pad2)
- added copper zone on B.Cu, net Net-(R18-Pad2)
Other:
- board text added: "+3V3"
- board text added: "+5V"
- board text added: "GND"
- board text added: "GNSS"
- board text added: "I"
- board text added: "O"
- board text added: "R+GB"
- board text added: "RX"
- board text added: "Radio"
- board text added: "TX"
- board text removed: "R + G B"
