File: KiCad Files/Alcantara_v.1.0.sch (KiCad schematic (older format))
At the start: 21 parts, among them IC3 TLV803EA30DCKR, J5 PJS008U-3000-0, J8 53261-0527, Q1 MMSS8050-H-TP, Q2 MMSS8050-H-TP

Commit message: Origanized Folders
Connections:
- no-connect marks 43 -> 10
Other:
- note removed: "> 4 camadas go BRRRRRRRR"
- note removed: "> Conferir o pinout dos botões de EN e IO0"
- note removed: "> Editar silk dos botões"
- note removed: "> Escolher uma chave deslizante para o liga/desliga"
- note removed: "> Mover o capacitor e resistor de reset mais pra perto\n da ESP"
- note removed: "> Mudar o conector micro USB para um 100% SMD"
- note removed: "> Ou ligar junto ao RGB principal"
- note removed: "> Ponderar sobre a possibilidade de retirar os LEDs do FTDI"
- note removed: ">Refletir sobre quais decisões me trouxeram até aqui"
- note removed: "LISTA DE AFAZERES"
- moved on the sheet: C1, C2, C3, J5, MOD1, R13, R26, R3, R5

Commit message: Added Images
Other:
- note added: "Boot Button"
- note added: "External Picoblade\n"
- note added: "If there is any trouble reading pins,\ncheck the internal pull resistors,\nthey vary with every pin."
- note added: "Peripherals"
- note added: "Pin 12 (GPS_ON_OFF) may need to have a pull-up or a pull-down\nressitor depending on the ESP internal flash.\nNote that the pull-down resistors are in the "Tecommunications"\npage on the gate of the Mosfet that actuates the GPS.\n\nThis is needed because pin 12 is a bootstrap pin, used to select the\ninternal flash voltage: \n1 -> 1.8V\n0 -> 3.3V\n\nIf a 3.3V flash is used (standard) use the Mosf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"
- note added: "Power"
- note added: "Read about the pull-up\nresitors for SD cards here:\nhttps://electronics.stackex\nchange.com/questions/39\n571/how-to-do-pulling-up\n-or-down-correctly-when-\ninterfacing-a-microsd-card"
- note added: "Reset Button"
- note added: "SD Card"
- note added: "Telecommunications"
- note removed: "Botão de Boot"
- note removed: "Botão de Reset\n"
- note removed: "Cartão SD"
- note removed: "Internal Pull-down"
- note removed: "Internal Pull-up"
- note removed: "Ler aqui sobre os resistores de pull-up para cartões SD:\nhttps://electronics.stackexchange.com/questions/39571/how-to-\ndo-pulling-up-or-down-correctly-when-interfacing-a-microsd-card"
- note removed: "Os resistores de pull-up ou pull-down devem ser utilizados um\npor vez, dependendo da tensão da flash interna da ESP.\nNote que os resistores que atuam como pull-down estão na\npágina "Tecommunications" pois lá eles são os resistores do\nMosfet que aciona o GPS.\n\nIsso ocorre pois o pino 12 é um pino lido no boot para selecionar\na tensão que alimenta a flash interna: \n1 -> 1.8V\n0 -> 3.3V\n\nS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"
- note removed: "Picoblade Externo\n"
- note removed: "Verificar que os pinos conectados em VP e VN não flutuarão, \nse não um pullup será necessário nesses pinos. Ele não possui\npullup interno."
- moved on the sheet: C1, C2, C3, C4, C5, IC3, J5, J8, MOD1, Q1, Q2, R1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
