File: KiCad Files/Power Management.sch (KiCad schematic (older format))
At the start: 25 parts, among them IC1 TLV809ED29DBZR, IC2 MAX17201G+T, Q4 Q_PMOS_GSD, U2 TPS61092, U3 LD1117S33TR_SOT223

Commit message: Added Images
Other:
- note added: "The MAX17201 is an I2C single cell battery monitor. Be aware of \nthe differences of the MAX17211, wich uses the 1-Wire protocol.\n\nThis component will measure the battery volatge and with the\n0.01 ohm shunt it will also measure the current.\n\nAlso be aware of the MAX17205, wich is a multiple cell monitor."
- note added: "The P channel Mosfet in series with the batery works as a\nsimple reverse polarity protection circuit.\n\nIf the battery is reversed it will not conduct, hence not turning the\ncircuit on.\n\nI didin't use the zenner on the gate because the Mosfet's maximum\nVgs voltage is higher than what we will be applied by the battery.\n\nAlso, I didin't use a resistor on the gate because the mosfet is \ncon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"
- note added: "The TLV809ED29DBZR is a voltage supervisor with a push-pull output.\nWhen its input voltage goes above the threshold of 2.93V it takes its output to VCC, enabling the Boost Converter. \nWhen VDD falls bellow the threshold its outut is pulled to 0V, turning the system off.\nThis protects the battery from undervolting damage."
- note removed: "O Mosfet tipo P em série com a bateria faz a função de\nproteção contra polaridade reversa.\n\nCaso a bateria seja invertida ele não conduzirá, protegendo\no circuito.\n\nNão utilizei um zener pois a tensão Vgs máxima permitida\nestá acima da que submeteremos no mosfet.\n\nAlém disso, descartei a necessidade de utilizar um resistor\nno gate, pois esse mosfet ficará constantemente ligado,\nentão o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"
- note removed: "O componente MAX17201 é um monitor de bateria\nde célula única via I2C. Atentar para a diferença com\no MAX17211, que utiliza o protocolo 1-Wire.\n\nEste componente vai fornecer dados como a corrente que flui\npela bateria (por meio do shunt de 0.01ohm) e a tensão nela.\n\nAtentar-se também sobre a diferença com o MAX17205,\nque é um monitor para múltiplas células."
- note removed: "O componente TLV809ED29DBZR é um surpervisor de tensão com saída push-pull.\nQuando a tensão de alimentação está acima do seu threshold de 2.93V ele leva a sua saída a VCC, habilitando o Boost Converter. \nCaso a tensão em VDD caia abaixo do seu threshold a saída será puxada para 0V, desligando o sistema"
- note removed: "Retirei os resistores de 150ohms em série com os pinos SDA e SCL antes dos pullup"
- moved on the sheet: BT2, C7, C9, IC2, Q4, R10, R12, R14, R15, R16, R7, R9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
