File: KiCad Files/Telecommunications.sch (KiCad schematic (older format))
At the start: 18 parts, among them J1 U_FL-R-SMT_10_, J2 142-0701-801, J3 142-0701-801, Q7 2N7002NXAKR, U1 E22-900M30S, U4 NEO-M8N

Commit message: Added Images
Other:
- note added: "The Mosfet is used for turning the Neo-M8N on or off completely, enabling a low power mode for the board.\nThe module offers alternatives for low power modes via commands, but the documentation is rubbish.\nSHAME on u-blox for not making an enable pin, SHAME >:C"
- moved on the sheet: BT1, C13, C14, C15, C21, D1, J1, J2, J3, L2, Q7, R11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
