File: KiCad_Files/Peripherals.sch (KiCad schematic (older format))
At the start: 24 parts, among them J4 USB_B_Micro, Q3 2N7002NXAKR, U5 Buzzer_SMD_AST0760MCTRQ, U6 USBLC6-2SC6, U7 FT232RL-REEL

Commit message: Add shapes 3D folder
Now all 3D models for the components are stored in a single folder, thanks to the Archive Plugin from https://github.com/MitjaNemec/Kicad_action_plugins.git
Parts:
- C16, C17, C18, C19, C20: symbol Device:C_Small -> archive:Device_C_Small
- D2: symbol Device:LED_RGBA -> archive:Device_LED_RGBA
- J4: symbol Connector:USB_B_Micro -> archive:Connector_USB_B_Micro
- Q3: symbol SamacSys_Parts:2N7002NXAKR -> archive:SamacSys_Parts_2N7002NXAKR
- R19, R20, R21, R22, R23, R24, R25, R27, R28, R30, R31: symbol Device:R_Small -> archive:Device_R_Small
- S1, S2: symbol SamacSys_Parts:KSC941JLFS -> archive:SamacSys_Parts_KSC941JLFS
- U5: symbol SamacSys_Parts:Buzzer_SMD_AST0760MCTRQ -> archive:SamacSys_Parts_Buzzer_SMD_AST0760MCTRQ
- U6: symbol Power_Protection:USBLC6-2SC6 -> archive:Power_Protection_USBLC6-2SC6
- U7: symbol dk_Interface-Controllers:FT232RL-REEL -> archive:dk_Interface-Controllers_FT232RL-REEL
Changed lines of the file:
@@
 $EndDescr
 $Comp
-L dk_Interface-Controllers:FT232RL-REEL U?
+L archive:dk_Interface-Controllers_FT232RL-REEL U?
 U 1 1 60D8D886
 P 9500 3450
@@
 $EndComp
 $Comp
-L Connector:USB_B_Micro J4
+L archive:Connector_USB_B_Micro J4
 U 1 1 60E1BC52
 P 2300 1900
@@
 NoConn ~ 2200 2300
 $Comp
-L power:GND #PWR035
+L archive:power_GND #PWR035
 U 1 1 60E2020B
 P 2300 2350
@@
 	2300 2350 2300 2300
 $Comp
-L Device:R_Small R27
+L archive:Device_R_Small R27
 U 1 1 60E207DE
 P 8000 3150
@@
 $EndComp
 $Comp
-L Device:R_Small R28
+L archive:Device_R_Small R28
 U 1 1 60E21E35
 P 8000 3550
@@
 $EndComp
 $Comp
-L power:GND #PWR044
+L archive:power_GND #PWR044
 U 1 1 60E2207D
 P 8000 3700
@@
 	8000 3350 8000 3250
 $Comp
-L Power_Protection:USBLC6-2SC6 U6
+L archive:Power_Protection_USBLC6-2SC6 U6
 U 1 1 60E25ED4
 P 4550 1850
@@
 	8000 2900 8000 3050
 $Comp
-L Device:C_Small C18
+L archive:Device_C_Small C18
 U 1 1 60E31E88
 P 10200 3350
@@
 $EndComp
 $Comp
-L power:GND #PWR050
+L archive:power_GND #PWR050
 U 1 1 60E335D5
 P 10550 3500
@@
 	10100 3350 9900 3350
 $Comp
-L power:+5V #PWR048
+L archive:power_+5V #PWR048
 U 1 1 60E33F83
 P 9650 2400
@@
 	9650 2450 9650 2400
 $Comp
-L power:+3V3 #PWR045
+L archive:power_+3V3 #PWR045
 U 1 1 60E34BD6
 P 9050 2400
@@
 	9300 2450 9300 2950
 $Comp
-L power:GND #PWR049
+L archive:power_GND #PWR049
 U 1 1 60E35BEC
 P 9650 2800
@@
 $EndComp
 $Comp
-L power:GND #PWR046
+L archive:power_GND #PWR046
 U 1 1 60E361F1
 P 9050 2800
@@
 $EndComp
 $Comp
-L Device:C_Small C17
+L archive:Device_C_Small C17
 U 1 1 60E370A2
 P 9650 2600
@@
 $EndComp
 $Comp
-L Device:C_Small C16
+L archive:Device_C_Small C16
 U 1 1 60E375B9
 P 9050 2600
@@
 FTDI_TX
 $Comp
-L power:GND #PWR047
+L archive:power_GND #PWR047
 U 1 1 60F952ED
 P 9450 4950
@@
 USB to Serial Converter
 $Comp
-L Device:R_Small R?
+L archive:Device_R_Small R?
 U 1 1 6101D387
 P 2050 4550
@@
 $EndComp
 $Comp
-L Device:R_Small R?
+L archive:Device_R_Small R?
 U 1 1 6101D38D
 P 2050 4350
@@
 $EndComp
 $Comp
-L Device:R_Small R?
+L archive:Device_R_Small R?
 U 1 1 6101D393
 P 2050 4150
@@
 RGB_LED_B
 $Comp
-L Device:R_Small R24
+L archive:Device_R_Small R24
 U 1 1 61029512
 P 4850 4600
@@
 	4950 4600 5050 4600
 $Comp
-L Device:R_Small R25
+L archive:Device_R_Small R25
 U 1 1 6102A606
 P 5050 4800
@@
 	5050 4950 5050 4900
 $Comp
-L power:GND #PWR041
+L archive:power_GND #PWR041
 U 1 1 6102C851
 P 5450 5050
@@
 Connection ~ 5450 4950
 $Comp
-L power:+5V #PWR040
+L archive:power_+5V #PWR040
 U 1 1 6102E81A
 P 5450 3600
@@
 	4650 4600 4750 4600
 $Comp
-L power:GND #PWR037
+L archive:power_GND #PWR037
 U 1 1 61048D66
 P 3250 7050
@@
 $EndComp
 $Comp
-L Device:R_Small R19
+L archive:Device_R_Small R19
 U 1 1 6104E8B6
 P 1950 6700
@@
 	1950 6800 1950 6850
 $Comp
-L power:+3V3 #PWR033
+L archive:power_+3V3 #PWR033
 U 1 1 610509F0
 P 1950 6550
@@
 	1950 6550 1950 6600
 $Comp
-L Device:R_Small R23
+L archive:Device_R_Small R23
 U 1 1 610556C6
 P 5100 6700
@@
 	5100 6800 5100 6850
 $Comp
-L power:+3V3 #PWR038
+L archive:power_+3V3 #PWR038
 U 1 1 610556CE
 P 5100 6550
@@
 FTDI_RTS
 $Comp
-L power:GND #PWR055
+L archive:power_GND #PWR055
 U 1 1 614ABBBD
 P 4550 2300
@@
 	4550 2300 4550 2250
 $Comp
-L power:+3V3 #PWR054
+L archive:power_+3V3 #PWR054
 U 1 1 614AEBD0
 P 4550 1400
@@
 	4550 1400 4550 1450
 $Comp
-L Device:R_Small R31
+L archive:Device_R_Small R31
 U 1 1 60E15770
 P 4800 6850
@@
 	4900 6850 5100 6850
 $Comp
-L Device:C_Small C20
+L archive:Device_C_Small C20
 U 1 1 60E2260F
 P 4550 7000
@@
 	4550 6850 4250 6850
 $Comp
-L power:GND #PWR057
+L archive:power_GND #PWR057
 U 1 1 60E25191
 P 4550 7150
@@
 	4550 7150 4550 7100
 $Comp
-L Device:R_Small R30
+L archive:Device_R_Small R30
 U 1 1 60E29CED
 P 1700 6850
@@
 	1800 6850 1950 6850
 $Comp
-L Device:C_Small C19
+L archive:Device_C_Small C19
 U 1 1 60E2A26E
 P 1450 7000
@@
 	1450 6850 1600 6850
 $Comp
-L power:GND #PWR056
+L archive:power_GND #PWR056
 U 1 1 60E2D0D4
 P 1450 7150
@@
 	1450 7150 1450 7100
 $Comp
-L Device:LED_RGBA D2
+L archive:Device_LED_RGBA D2
 U 1 1 60F72337
 P 1550 4350
@@
 $EndComp
 $Comp
-L power:+3V3 #PWR0102
+L archive:power_+3V3 #PWR0102
 U 1 1 60F808B6
 P 1050 4000
@@
 	6400 6850 6400 7050
 $Comp
-L power:GND #PWR042
+L archive:power_GND #PWR042
 U 1 1 610461A3
 P 6400 7050
@@
 $EndComp
 $Comp
-L SamacSys_Parts:KSC941JLFS S1
+L archive:SamacSys_Parts_KSC941JLFS S1
 U 1 1 60F54AAA
 P 2500 7450
@@
 	2300 4150 2150 4150
 $Comp
-L SamacSys_Parts:2N7002NXAKR Q3
+L archive:SamacSys_Parts_2N7002NXAKR Q3
 U 1 1 615A524B
 P 5150 4600
@@
 $EndComp
 $Comp
-L SamacSys_Parts:Buzzer_SMD_AST0760MCTRQ U5
+L archive:SamacSys_Parts_Buzzer_SMD_AST0760MCTRQ U5
 U 1 1 615A94E9
 P 5450 3900
@@
 Connection ~ 5100 6850
 $Comp
-L SamacSys_Parts:KSC941JLFS S2
+L archive:SamacSys_Parts_KSC941JLFS S2
 U 1 1 60F919E7
 P 5650 7450

Commit message: Realocated and replaced components
Components where replaced because of the chip shortage, such as the 3.3 V Voltage regulator, the USB ESD protector and the SD Card holder.

The ESP32 has been rotated and moved closer to the center of the board, now having it's antenna positioned outside of the original board outline, providing better range for the Bluetooth and Wi-Fi.
Parts:
- removed U6: USBLC6-2SC6, Package_TO_SOT_SMD:SOT-23-6, symbol archive:Power_Protection_USBLC6-2SC6
- added IC5: PESD2ETH-ADX, SamacSys_Parts:SOT95P275X110-6N, symbol SamacSys_Parts:PESD2ETH-ADX
Connections:
- net +3V3: now also IC5.5
- net GND: now also IC5.2
- net USB_CONN_D+: now also IC5.6
- net USB_CONN_D-: now also IC5.4
- net USB_D+: now also IC5.1
- net USB_D-: now also IC5.3
- net at R23.1, R31.1, S2.4 (NO_2): now also S2.3 (NO_1)
- no-connect marks 14 -> 13
Changed lines of the file:
@@
 Wire Wire Line
 	8000 3350 8000 3250
-$Comp
-L archive:Power_Protection_USBLC6-2SC6 U6
-U 1 1 60E25ED4
-P 4550 1850
-F 0 "U6" H 4700 2400 50  0000 C CNN
-F 1 "USBLC6-2SC6" H 4950 2250 50  0000 C CNN
-F 2 "Package_TO_SOT_SMD:SOT-23-6" H 4550 1350 50  0001 C CNN
-F 3 "https://www.st.com/resource/en/datasheet/usblc6-2.pdf" H 4750 2200 50  0001 C CNN
-	1    4550 1850
-	1    0    0    -1
-$EndComp
 Text GLabel 2600 1700 2    50   Input ~ 0
 USB_CONN_V+
@@
 Text GLabel 2600 2000 2    50   Input ~ 0
 USB_CONN_D-
-Text GLabel 4150 1750 0    50   Input ~ 0
+Text GLabel 4250 1625 0    50   Input ~ 0
 USB_CONN_D+
-Text GLabel 4950 1750 2    50   Input ~ 0
+Text GLabel 5150 1625 2    50   Input ~ 0
 USB_CONN_D-
-Text GLabel 4150 1950 0    50   Input ~ 0
+Text GLabel 4250 2125 0    50   Input ~ 0
 USB_D+
-Text GLabel 4950 1950 2    50   Input ~ 0
+Text GLabel 5150 2125 2    50   Input ~ 0
 USB_D-
 Wire Wire Line
@@
 L archive:power_GND #PWR055
 U 1 1 614ABBBD
-P 4550 2300
-F 0 "#PWR055" H 4550 2050 50  0001 C CNN
-F 1 "GND" H 4555 2127 50  0000 C CNN
-F 2 "" H 4550 2300 50  0001 C CNN
-F 3 "" H 4550 2300 50  0001 C CNN
-	1    4550 2300
-	1    0    0    -1
-$EndComp
-Wire Wire Line
-	4550 2300 4550 2250
+P 4700 2325
+F 0 "#PWR055" H 4700 2075 50  0001 C CNN
+F 1 "GND" H 4705 2152 50  0000 C CNN
+F 2 "" H 4700 2325 50  0001 C CNN
+F 3 "" H 4700 2325 50  0001 C CNN
+	1    4700 2325
+	1    0    0    -1
+$EndComp
+Wire Wire Line
+	4700 2325 4700 2275
 $Comp
 L archive:power_+3V3 #PWR054
 U 1 1 614AEBD0
-P 4550 1400
-F 0 "#PWR054" H 4550 1250 50  0001 C CNN
-F 1 "+3V3" H 4565 1573 50  0000 C CNN
-F 2 "" H 4550 1400 50  0001 C CNN
-F 3 "" H 4550 1400 50  0001 C CNN
-	1    4550 1400
-	1    0    0    -1
-$EndComp
-Wire Wire Line
-	4550 1400 4550 1450
+P 4700 1425
+F 0 "#PWR054" H 4700 1275 50  0001 C CNN
+F 1 "+3V3" H 4715 1598 50  0000 C CNN
+F 2 "" H 4700 1425 50  0001 C CNN
+F 3 "" H 4700 1425 50  0001 C CNN
+	1    4700 1425
+	1    0    0    -1
+$EndComp
+Wire Wire Line
+	4700 1425 4700 1475
 $Comp
 L archive:Device_R_Small R31
@@
 	0    -1   -1   0
 $EndComp
-NoConn ~ 5650 6250
 $Bitmap
 Pos 9125 6850
@@
 EndData
 $EndBitmap
+Wire Wire Line
+	4250 1625 4300 1625
+Wire Wire Line
+	4250 2125 4300 2125
+Wire Wire Line
+	5100 2125 5150 2125
+Wire Wire Line
+	5100 1625 5150 1625
+Wire Wire Line
+	5650 6250 5650 6150
+Wire Wire Line
+	5650 6150 5450 6150
+Wire Wire Line
+	5450 6150 5450 6850
+Connection ~ 5450 6850
+$Comp
+L SamacSys_Parts:PESD2ETH-ADX IC5
+U 1 1 625E745E
+P 4650 1725
+F 0 "IC5" H 5350 1990 50  0000 C CNN
+F 1 "PESD2ETH-ADX" H 5350 1899 50  0000 C CNN
+F 2 "SamacSys_Parts:SOT95P275X110-6N" H 5900 1825 50  0001 L CNN
+F 3 "https://assets.nexperia.com/documents/data-sheet/PESD2ETH-AD.pdf" H 5900 1725 50  0001 L CNN
+F 4 "Ultra low capacitance double rail-to-rail ESD protection diode" H 5900 1625 50  0001 L CNN "Description"
+F 5 "1.1" H 5900 1525 50  0001 L CNN "Height"
+F 6 "771-PESD2ETH-ADX" H 5900 1425 50  0001 L CNN "Mouser Part Number"
+F 7 "https://www.mouser.co.uk/ProductDetail/Nexperia/PESD2ETH-ADX?qs=W0yvOO0ixfHGl%2FIqaic%2F9w%3D%3D" H 5900 1325 50  0001 L CNN "Mouser Price/Stock"
+F 8 "Nexperia" H 5900 1225 50  0001 L CNN "Manufacturer_Name"
+F 9 "PESD2ETH-ADX" H 5900 1125 50  0001 L CNN "Manufacturer_Part_Number"
+	1    4650 1725
+	1    0    0    -1
+$EndComp
 $EndSCHEMATC

Commit message: Reduces board length to 101,5 mm
JLC PCB allows a 4 layer PCB to be manufactured for just $8,00 if it is within 102 x 102 mm. The previous version was 105,47 mm, making it cost $37,00.

To reduce the manufacturing cost the board had its size cut down to 101,5 mm. This was possible by moving the buzzer from the top left corner of the board to the free space between the two SMA connectors.
Parts:
- IC5: symbol SamacSys_Parts:PESD2ETH-ADX -> archive:SamacSys_Parts_PESD2ETH-ADX
Changed lines of the file:
@@
 Connection ~ 5450 6850
 $Comp
-L SamacSys_Parts:PESD2ETH-ADX IC5
+L archive:SamacSys_Parts_PESD2ETH-ADX IC5
 U 1 1 625E745E
 P 4650 1725
-F 0 "IC5" H 5350 1990 50  0000 C CNN
-F 1 "PESD2ETH-ADX" H 5350 1899 50  0000 C CNN
+F 0 "IC5" H 4800 1950 50  0000 C CNN
+F 1 "PESD2ETH-ADX" H 5075 1200 50  0000 C CNN
 F 2 "SamacSys_Parts:SOT95P275X110-6N" H 5900 1825 50  0001 L CNN
 F 3 "https://assets.nexperia.com/documents/data-sheet/PESD2ETH-AD.pdf" H 5900 1725 50  0001 L CNN
