File: KiCad_Files/Telecommunications.sch (KiCad schematic (older format))
At the start: 18 parts, among them J1 U_FL-R-SMT_10_, J2 142-0701-801, J3 142-0701-801, Q7 2N7002NXAKR, U1 E22-900M30S, U4 NEO-M8N

Commit message: Add shapes 3D folder
Now all 3D models for the components are stored in a single folder, thanks to the Archive Plugin from https://github.com/MitjaNemec/Kicad_action_plugins.git
Parts:
- BT1: symbol ML414H_IV01E:ML414H_IV01E -> archive:ML414H_IV01E_ML414H_IV01E
- C13, C14, C15, C21: symbol Device:C_Small -> archive:Device_C_Small
- D1: symbol Device:D_Schottky_Small -> archive:Device_D_Schottky_Small
- J1: symbol Alcantara_v.1.0-rescue:U_FL-R-SMT_10_-dk_Coaxial-Connectors-RF -> archive:Alcantara_v.1.0-rescue_U_FL-R-SMT_10_-dk_Coaxial-Connectors-RF
- J2, J3: symbol dk_Coaxial-Connectors-RF:142-0701-801 -> archive:dk_Coaxial-Connectors-RF_142-0701-801
- L2: symbol Device:L_Small -> archive:Device_L_Small
- Q7: symbol SamacSys_Parts:2N7002NXAKR -> archive:SamacSys_Parts_2N7002NXAKR
- R11, R17, R18, R33, R34: symbol Device:R_Small -> archive:Device_R_Small
- U1: symbol E22_Radios_Zenith:E22-900M30S -> archive:E22_Radios_Zenith_E22-900M30S
- U4: symbol Zenith_Modified_Libraries:NEO-M8N -> archive:Zenith_Modified_Libraries_NEO-M8N
Changed lines of the file:
@@
 	3425 2875 3425 2925
 $Comp
-L power:+3V3 #PWR019
+L archive:power_+3V3 #PWR019
 U 1 1 60E187D2
 P 2075 3275
@@
 $EndComp
 $Comp
-L power:GND #PWR020
+L archive:power_GND #PWR020
 U 1 1 60E19D9C
 P 2075 3675
@@
 $EndComp
 $Comp
-L Device:C_Small C13
+L archive:Device_C_Small C13
 U 1 1 60E1A4E4
 P 2075 3525
@@
 	2075 3625 2075 3675
 $Comp
-L dk_Coaxial-Connectors-RF:142-0701-801 J2
+L archive:dk_Coaxial-Connectors-RF_142-0701-801 J2
 U 1 1 60E543A4
 P 5250 4450
@@
 $EndComp
 $Comp
-L Device:L_Small L2
+L archive:Device_L_Small L2
 U 1 1 60E57109
 P 4400 3525
@@
 	4050 3225 4400 3225
 $Comp
-L Device:R_Small R18
+L archive:Device_R_Small R18
 U 1 1 60E5B23B
 P 3950 3225
@@
 $EndComp
 $Comp
-L Device:C_Small C15
+L archive:Device_C_Small C15
 U 1 1 60E5C8AF
 P 5250 3350
@@
 Connection ~ 4400 3225
 $Comp
-L Alcantara_v.1.0-rescue:U_FL-R-SMT_10_-dk_Coaxial-Connectors-RF J1
+L archive:Alcantara_v.1.0-rescue_U_FL-R-SMT_10_-dk_Coaxial-Connectors-RF J1
 U 1 1 60E666C0
 P 5250 3825
@@
 	9425 4600 9475 4600
 $Comp
-L power:+5V #PWR?
+L archive:power_+5V #PWR?
 U 1 1 60FC2EF1
 P 7525 4350
@@
 Connection ~ 7525 4500
 $Comp
-L power:GND #PWR?
+L archive:power_GND #PWR?
 U 1 1 60FC2EFC
 P 9525 4800
@@
 	9525 4700 9425 4700
 $Comp
-L power:GND #PWR?
+L archive:power_GND #PWR?
 U 1 1 60FC2F04
 P 8225 5150
@@
 	8225 4700 8325 4700
 $Comp
-L power:GND #PWR?
+L archive:power_GND #PWR?
 U 1 1 60FC2F0C
 P 7525 3800
@@
 	9425 4100 9475 4100
 $Comp
-L dk_Coaxial-Connectors-RF:142-0701-801 J?
+L archive:dk_Coaxial-Connectors-RF_142-0701-801 J?
 U 1 1 60FC2F34
 P 10525 3650
@@
 	6950 6500 6950 500
 $Comp
-L ML414H_IV01E:ML414H_IV01E BT?
+L archive:ML414H_IV01E_ML414H_IV01E BT?
 U 1 1 6116FC93
 P 2875 2625
@@
 $EndComp
 $Comp
-L Device:C_Small C14
+L archive:Device_C_Small C14
 U 1 1 61171146
 P 2825 2925
@@
 $EndComp
 $Comp
-L Device:R_Small R17
+L archive:Device_R_Small R17
 U 1 1 6117170F
 P 3125 2425
@@
 $EndComp
 $Comp
-L power:+3V3 #PWR022
+L archive:power_+3V3 #PWR022
 U 1 1 61172368
 P 3125 2025
@@
 $EndComp
 $Comp
-L power:GND #PWR021
+L archive:power_GND #PWR021
 U 1 1 61172B25
 P 2525 3025
@@
 	3125 2625 3075 2625
 $Comp
-L Device:D_Schottky_Small D1
+L archive:Device_D_Schottky_Small D1
 U 1 1 61179C6F
 P 3125 2175
@@
 GPS_TX
 $Comp
-L Device:R_Small R11
+L archive:Device_R_Small R11
 U 1 1 615FE2D1
 P 9525 3350
@@
 	9525 4000 9425 4000
 $Comp
-L power:+3V3 #PWR0115
+L archive:power_+3V3 #PWR0115
 U 1 1 61600D7D
 P 9525 3150
@@
 	9525 3150 9525 3250
 $Comp
-L Device:C_Small C21
+L archive:Device_C_Small C21
 U 1 1 61451F4E
 P 7525 4800
@@
 Connection ~ 7525 4600
 $Comp
-L E22_Radios_Zenith:E22-900M30S U1
+L archive:E22_Radios_Zenith_E22-900M30S U1
 U 1 1 612EA8AF
 P 8875 4150
@@
 $EndComp
 $Comp
-L power:GNDA #PWR0118
+L archive:power_GNDA #PWR0118
 U 1 1 616C88D8
 P 5250 3475
@@
 NoConn ~ 3925 4275
 $Comp
-L power:GNDA #PWR0119
+L archive:power_GNDA #PWR0119
 U 1 1 616F731D
 P 5250 4675
@@
 	4900 3825 5050 3825
 $Comp
-L power:GNDA #PWR0120
+L archive:power_GNDA #PWR0120
 U 1 1 61701EA3
 P 5250 4050
@@
 	4100 3925 3925 3925
 $Comp
-L power:GNDA #PWR0121
+L archive:power_GNDA #PWR0121
 U 1 1 6170C71A
 P 4100 3975
@@
 Connection ~ 4100 3925
 $Comp
-L Device:R_Small R?
+L archive:Device_R_Small R?
 U 1 1 61A3932D
 P 2625 5950
@@
 	2725 5950 2825 5950
 $Comp
-L Device:R_Small R?
+L archive:Device_R_Small R?
 U 1 1 61A39334
 P 2825 6150
@@
 	2825 6300 2825 6250
 $Comp
-L power:GND #PWR?
+L archive:power_GND #PWR?
 U 1 1 61A39340
 P 3225 6400
@@
 	2425 5950 2525 5950
 $Comp
-L SamacSys_Parts:2N7002NXAKR Q?
+L archive:SamacSys_Parts_2N7002NXAKR Q?
 U 1 1 61A39350
 P 2925 5950
@@
 NoConn ~ 4025 4575
 $Comp
-L Zenith_Modified_Libraries:NEO-M8N U?
+L archive:Zenith_Modified_Libraries_NEO-M8N U?
 U 1 1 60D8A4F2
 P 3225 4275
@@
 Connection ~ 3225 5300
 $Comp
-L power:GND1 #PWR0123
+L archive:power_GND1 #PWR0123
 U 1 1 61A77D8E
 P 2825 5500
@@
 Connection ~ 3125 5300
 $Comp
-L power:GND1 #PWR0124
+L archive:power_GND1 #PWR0124
 U 1 1 61A7BDEF
 P 3425 2925

Commit message: Change radio's decoupling capacitor to the 1206 packaging size.
Upgrades the radios capacitor and rerouted it's traces to better accommodate grounding vias.
Parts:
- C21: footprint Capacitor_SMD:C_0805_2012Metric -> Capacitor_SMD:C_1206_3216Metric
Changed lines of the file:
@@
 F 0 "C21" H 7617 4846 50  0000 L CNN
 F 1 "1uF" H 7617 4755 50  0000 L CNN
-F 2 "Capacitor_SMD:C_0805_2012Metric" H 7525 4800 50  0001 C CNN
+F 2 "Capacitor_SMD:C_1206_3216Metric" H 7525 4800 50  0001 C CNN
 F 3 "~" H 7525 4800 50  0001 C CNN
 	1    7525 4800
