File: KiCad_Files/Alcantara_v.1.0.kicad_pcb (KiCad board)
At the start: 4 copper layers, 101.5 x 43.6 mm, 90 parts, among them IC1 TLV809ED29DBZR, IC2 MAX17201G+T, IC3 TLV803EA30DCKR, IC4 TC1264-3.3VDB, IC5 PESD2ETH-ADX, J1 U_FL-R-SMT_10_, J2 142-0701-801, J3 142-0701-801, J4 USB_B_Micro, J5 MEM2075-00-140-01-A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

Commit message: Change radio's decoupling capacitor to the 1206 packaging size.
Upgrades the radios capacitor and rerouted it's traces to better accommodate grounding vias.
Parts:
- C21: footprint Capacitor_SMD:C_0805_2012Metric -> Capacitor_SMD:C_1206_3216Metric
- S6: footprint Downloaded:SW_MSS-102545-14A-V-SMT -> Alcantara_Footprints:SW_MSS-102545-14A-V-SMT
- turned C21 to 90 degrees
Routing:
- net +5V: track 178.1 -> 180.0 mm
- net GND: vias 224 -> 223

Commit message: Add MS5607 barometer.
Adds MS5607 barometer and reorganized silkscreen.
Parts:
- removed the G*** at (80.1, 62.9)
- removed the G*** at (108.2, 33.7)
- removed REF**: 2.4_GHZ_Antenna_Left_Art, LogosZenith:2.4_GHZ_Antenna_Left_Art
- added G***: LOGO, LogosZenith:Alcantara_1,7mm, B.Cu at (80.2, 61.6)
- added G***: LOGO, LogosZenith:Logo_15,9mm, F.Cu at (125.8, 25.9)
- added U3: MS560702BA03-50, digikey-footprints:SMD-8_5x3mm, B.Cu at (109.1, 33.2)
Routing:
- net GND: track 75.7 -> 93.1 mm, vias 223 -> 221
- net +3V3: track 75.3 -> 81.0 mm, vias 30 -> 33
- net GAUGE_SCL: track 65.0 -> 66.8 mm
- net GAUGE_SDA: track 64.5 -> 65.9 mm
- net EN: track 65.3 -> 64.1 mm
- net IO0: track 83.4 -> 82.3 mm
Other:
- board text added: "By Júlio Calandrin :)"
