File: KiCad_Files/Power Management.sch (KiCad schematic (older format))
At the start: 25 parts, among them IC1 TLV809ED29DBZR, IC2 MAX17201G+T, Q4 Q_PMOS_GSD, U2 TPS61092, U3 LD1117S33TR_SOT223

Commit message: Add shapes 3D folder
Now all 3D models for the components are stored in a single folder, thanks to the Archive Plugin from https://github.com/MitjaNemec/Kicad_action_plugins.git
Parts:
- BT2: symbol Device:Battery_Cell -> archive:Device_Battery_Cell
- C10: symbol Device:CP_Small -> archive:Device_CP_Small
- C11, C12, C6, C7, C8, C9: symbol Device:C_Small -> archive:Device_C_Small
- IC1: symbol SamacSys_Parts:TLV809ED29DBZR -> archive:SamacSys_Parts_TLV809ED29DBZR
- IC2: symbol SamacSys_Parts:MAX17201G+T -> archive:SamacSys_Parts_MAX17201G+T
- L1: symbol Device:L_Small -> archive:Device_L_Small
- Q4: symbol Device:Q_PMOS_GSD -> archive:Device_Q_PMOS_GSD
- R10, R12, R14, R15, R16, R29, R8, R9: symbol Device:R_Small -> archive:Device_R_Small
- R7: symbol Device:R -> archive:Device_R
- S6: symbol MSS-102545-14A-V-SMT:MSS-102545-14A-V-SMT -> archive:MSS-102545-14A-V-SMT_MSS-102545-14A-V-SMT
- TH1: symbol Device:Thermistor_NTC -> archive:Device_Thermistor_NTC
- U2: symbol Regulator_Switching:TPS61092 -> archive:Regulator_Switching_TPS61092
- U3: symbol Regulator_Linear:LD1117S33TR_SOT223 -> archive:Regulator_Linear_LD1117S33TR_SOT223
Changed lines of the file:
@@
 $EndDescr
 $Comp
-L power:GND #PWR012
+L archive:power_GND #PWR012
 U 1 1 60D85621
 P 6650 3825
@@
 Pack
 $Comp
-L Device:Thermistor_NTC TH?
+L archive:Device_Thermistor_NTC TH?
 U 1 1 60D8563E
 P 5550 3325
@@
 $EndComp
 $Comp
-L Device:R R7
+L archive:Device_R R7
 U 1 1 60D85651
 P 6250 3725
@@
 	7200 2575 8050 2575
 $Comp
-L Device:R_Small R?
+L archive:Device_R_Small R?
 U 1 1 60D8567C
 P 7350 1875
@@
 $EndComp
 $Comp
-L Device:R_Small R?
+L archive:Device_R_Small R?
 U 1 1 60D85683
 P 8050 1875
@@
 $EndComp
 $Comp
-L Device:R_Small R?
+L archive:Device_R_Small R?
 U 1 1 60D85689
 P 7700 1875
@@
 $EndComp
 $Comp
-L Device:R_Small R?
+L archive:Device_R_Small R?
 U 1 1 60D85697
 P 8450 2175
@@
 Connection ~ 7700 1675
 $Comp
-L power:+3V3 #PWR?
+L archive:power_+3V3 #PWR?
 U 1 1 60D856B4
 P 7700 1575
@@
 $EndComp
 $Comp
-L Regulator_Linear:LD1117S33TR_SOT223 U3
+L archive:Regulator_Linear_LD1117S33TR_SOT223 U3
 U 1 1 60D979F1
 P 9100 5400
@@
 $EndComp
 $Comp
-L Device:C_Small C9
+L archive:Device_C_Small C9
 U 1 1 60D9A0A0
 P 5150 2375
@@
 $EndComp
 $Comp
-L Device:C_Small C7
+L archive:Device_C_Small C7
 U 1 1 60D9AA24
 P 7300 3375
@@
 $EndComp
 $Comp
-L Device:C_Small C11
+L archive:Device_C_Small C11
 U 1 1 60DA450D
 P 8500 5700
@@
 $EndComp
 $Comp
-L Device:C_Small C12
+L archive:Device_C_Small C12
 U 1 1 60DA4E3C
 P 9650 5700
@@
 $EndComp
 $Comp
-L power:GND #PWR016
+L archive:power_GND #PWR016
 U 1 1 60DA5F25
 P 9100 6000
@@
 	9100 5700 9100 6000
 $Comp
-L power:GND #PWR015
+L archive:power_GND #PWR015
 U 1 1 60DAA209
 P 8500 6000
@@
 $EndComp
 $Comp
-L power:GND #PWR017
+L archive:power_GND #PWR017
 U 1 1 60DAA5AA
 P 9650 6000
@@
 	8500 5400 8800 5400
 $Comp
-L power:+3V3 #PWR018
+L archive:power_+3V3 #PWR018
 U 1 1 60DB2DA4
 P 9900 5250
@@
 Connection ~ 9650 5400
 $Comp
-L Device:R_Small R?
+L archive:Device_R_Small R?
 U 1 1 60DF3D23
 P 5600 1925
@@
 	3700 5350 3800 5350
 $Comp
-L Device:C_Small C6
+L archive:Device_C_Small C6
 U 1 1 60E78225
 P 1250 6200
@@
 Connection ~ 4750 5350
 $Comp
-L Device:C_Small C8
+L archive:Device_C_Small C8
 U 1 1 60EDD3EF
 P 5250 5600
@@
 	5250 5500 5250 5350
 $Comp
-L power:GND #PWR09
+L archive:power_GND #PWR09
 U 1 1 60EE21CD
 P 5250 5800
@@
 	5250 5800 5250 5700
 $Comp
-L Device:CP_Small C10
+L archive:Device_CP_Small C10
 U 1 1 60EE6DA6
 P 5700 5600
@@
 Connection ~ 5250 5350
 $Comp
-L power:GND #PWR011
+L archive:power_GND #PWR011
 U 1 1 60EEBF1A
 P 5700 5800
@@
 	5700 5800 5700 5700
 $Comp
-L power:+5V #PWR010
+L archive:power_+5V #PWR010
 U 1 1 60EF0BEA
 P 5700 5200
@@
 Connection ~ 5700 5350
 $Comp
-L power:+5V #PWR014
+L archive:power_+5V #PWR014
 U 1 1 60EF9622
 P 8500 5250
@@
 Stand-alone Fuel Gauge
 $Comp
-L Device:Battery_Cell BT2
+L archive:Device_Battery_Cell BT2
 U 1 1 61591953
 P 4050 2725
@@
 $EndComp
 $Comp
-L power:GND #PWR0101
+L archive:power_GND #PWR0101
 U 1 1 6100DB47
 P 4400 6800
@@
 Connection ~ 4300 6550
 $Comp
-L Device:Q_PMOS_GSD Q4
+L archive:Device_Q_PMOS_GSD Q4
 U 1 1 610D18A9
 P 4650 1275
@@
 $EndComp
 $Comp
-L power:GND #PWR0108
+L archive:power_GND #PWR0108
 U 1 1 610FCF6D
 P 4650 1575
@@
 $EndComp
 $Comp
-L Regulator_Switching:TPS61092 U2
+L archive:Regulator_Switching_TPS61092 U2
 U 1 1 60DF7C3A
 P 4200 5850
@@
 	1000 5650 1250 5650
 $Comp
-L Device:L_Small L1
+L archive:Device_L_Small L1
 U 1 1 60E6B8CB
 P 3150 5350
@@
 	1250 5350 1250 5650
 $Comp
-L power:GND #PWR0109
+L archive:power_GND #PWR0109
 U 1 1 612ACFAF
 P 1250 6800
@@
 $EndComp
 $Comp
-L power:GND #PWR0110
+L archive:power_GND #PWR0110
 U 1 1 612B0FCE
 P 3700 6800
@@
 	2900 6800 2900 6550
 $Comp
-L power:GND #PWR0111
+L archive:power_GND #PWR0111
 U 1 1 612ACC1E
 P 2900 6800
@@
 $EndComp
 $Comp
-L SamacSys_Parts:TLV809ED29DBZR IC1
+L archive:SamacSys_Parts_TLV809ED29DBZR IC1
 U 1 1 612EBEE6
 P 3400 6200
@@
 $EndComp
 $Comp
-L Device:R_Small R?
+L archive:Device_R_Small R?
 U 1 1 60D85691
 P 5550 2925
@@
 $EndComp
 $Comp
-L SamacSys_Parts:MAX17201G+T IC2
+L archive:SamacSys_Parts_MAX17201G+T IC2
 U 1 1 613217CA
 P 5800 2325
@@
 	5900 3725 4050 3725
 $Comp
-L power:GND #PWR0112
+L archive:power_GND #PWR0112
 U 1 1 61366CA9
 P 5550 3475
@@
 Connection ~ 5550 3125
 $Comp
-L power:GND #PWR0113
+L archive:power_GND #PWR0113
 U 1 1 61376F3D
 P 5150 2575
@@
 	7300 3125 7200 3125
 $Comp
-L power:GND #PWR0114
+L archive:power_GND #PWR0114
 U 1 1 6138DA91
 P 7300 3825
@@
 	4650 1475 4650 1575
 $Comp
-L MSS-102545-14A-V-SMT:MSS-102545-14A-V-SMT S6
+L archive:MSS-102545-14A-V-SMT_MSS-102545-14A-V-SMT S6
 U 1 1 6196346E
 P 2125 6100
@@
 	1775 5650 3800 5650
 $Comp
-L Device:R_Small R?
+L archive:Device_R_Small R?
 U 1 1 61991C9D
 P 1600 5975
@@
 	1600 6200 1825 6200
 $Comp
-L Device:R_Small R?
+L archive:Device_R_Small R?
 U 1 1 6199CCDA
 P 1600 6400
@@
 Connection ~ 1600 6200
 $Comp
-L power:GND #PWR0106
+L archive:power_GND #PWR0106
 U 1 1 619A465D
 P 1600 6800

Commit message: Realocated and replaced components
Components where replaced because of the chip shortage, such as the 3.3 V Voltage regulator, the USB ESD protector and the SD Card holder.

The ESP32 has been rotated and moved closer to the center of the board, now having it's antenna positioned outside of the original board outline, providing better range for the Bluetooth and Wi-Fi.
Parts:
- removed C11: 0.1uF, Capacitor_SMD:C_1206_3216Metric, symbol archive:Device_C_Small
- removed U3: LD1117S33TR_SOT223, Package_TO_SOT_SMD:SOT-223-3_TabPin2, symbol archive:Regulator_Linear_LD1117S33TR_SOT223
- added IC4: TC1264-3.3VDB, SamacSys_Parts:SOT230P700X180-4N, symbol SamacSys_Parts:TC1264-3.3VDB
Connections:
- net +3V3: now also IC4.3 (VOUT)
- net +5V: now also IC4.1 (VIN)
- net GND: now also IC4.2 (GND_1), IC4.4 (GND_2)
- net Pack: now also S6.2; no longer S6.3
- net at R29.2, R8.1: now also S6.3; no longer S6.2
Other:
- note added: "The MAX17201 is an I2C single cell battery monitor. Be aware of \nthe differences of the MAX17211, wich uses the 1-Wire protocol.\n\nThis component will measure the battery voltage and using a\n0.01 ohm shunt it will also measure the current.\n\nAlso be aware of the MAX17205, wich is a multiple cell monitor."
- note added: "The P channel Mosfet in series with the batery works as a\nsimple reverse polarity protection circuit.\n\nIf the battery is reversed it will not conduct, hence not turning the\ncircuit on.\n\nI didin't use the zenner on the gate because the Mosfet's maximum\nVgs voltage is higher than what will be applied by the battery.\n\nAlso, I didin't use a resistor on the gate because the mosfet is \nconsta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"
- note added: "There's no capacitor in the input\nbecause C10 and C8 are placed\nnear the regulator on the PCB."
- note removed: "The MAX17201 is an I2C single cell battery monitor. Be aware of \nthe differences of the MAX17211, wich uses the 1-Wire protocol.\n\nThis component will measure the battery volatge and with the\n0.01 ohm shunt it will also measure the current.\n\nAlso be aware of the MAX17205, wich is a multiple cell monitor."
- note removed: "The P channel Mosfet in series with the batery works as a\nsimple reverse polarity protection circuit.\n\nIf the battery is reversed it will not conduct, hence not turning the\ncircuit on.\n\nI didin't use the zenner on the gate because the Mosfet's maximum\nVgs voltage is higher than what we will be applied by the battery.\n\nAlso, I didin't use a resistor on the gate because the mosfet is \ncon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"
- moved on the sheet: C12
Changed lines of the file:
@@
-$EndComp
-$Comp
-L archive:Regulator_Linear_LD1117S33TR_SOT223 U3
-U 1 1 60D979F1
-P 9100 5400
-F 0 "U3" H 9100 5642 50  0000 C CNN
-F 1 "LD1117S33TR_SOT223" H 9100 5551 50  0000 C CNN
-F 2 "Package_TO_SOT_SMD:SOT-223-3_TabPin2" H 9100 5600 50  0001 C CNN
-F 3 "http://www.st.com/st-web-ui/static/active/en/resource/technical/document/datasheet/CD00000544.pdf" H 9200 5150 50  0001 C CNN
-	1    9100 5400
-	1    0    0    -1
 $EndComp
 $Comp
@@
 $EndComp
 $Comp
-L archive:Device_C_Small C11
-U 1 1 60DA450D
-P 8500 5700
-F 0 "C11" H 8550 5800 50  0000 L CNN
-F 1 "0.1uF" H 8550 5600 50  0000 L CNN
-F 2 "Capacitor_SMD:C_1206_3216Metric" H 8500 5700 50  0001 C CNN
-F 3 "~" H 8500 5700 50  0001 C CNN
-	1    8500 5700
-	1    0    0    -1
-$EndComp
-$Comp
 L archive:Device_C_Small C12
 U 1 1 60DA4E3C
-P 9650 5700
-F 0 "C12" H 9700 5800 50  0000 L CNN
-F 1 "10uF" H 9700 5600 50  0000 L CNN
-F 2 "Capacitor_SMD:C_1206_3216Metric" H 9650 5700 50  0001 C CNN
-F 3 "~" H 9650 5700 50  0001 C CNN
-	1    9650 5700
+P 9950 5675
+F 0 "C12" H 10000 5775 50  0000 L CNN
+F 1 "10uF" H 10000 5575 50  0000 L CNN
+F 2 "Capacitor_SMD:C_1206_3216Metric" H 9950 5675 50  0001 C CNN
+F 3 "~" H 9950 5675 50  0001 C CNN
+	1    9950 5675
 	1    0    0    -1
 $EndComp
@@
 	1    0    0    -1
 $EndComp
-Wire Wire Line
-	9100 5700 9100 6000
-$Comp
-L archive:power_GND #PWR015
-U 1 1 60DAA209
-P 8500 6000
-F 0 "#PWR015" H 8500 5750 50  0001 C CNN
-F 1 "GND" H 8505 5827 50  0000 C CNN
-F 2 "" H 8500 6000 50  0001 C CNN
-F 3 "" H 8500 6000 50  0001 C CNN
-	1    8500 6000
-	1    0    0    -1
-$EndComp
 $Comp
 L archive:power_GND #PWR017
 U 1 1 60DAA5AA
-P 9650 6000
-F 0 "#PWR017" H 9650 5750 50  0001 C CNN
-F 1 "GND" H 9655 5827 50  0000 C CNN
-F 2 "" H 9650 6000 50  0001 C CNN
-F 3 "" H 9650 6000 50  0001 C CNN
-	1    9650 6000
-	1    0    0    -1
-$EndComp
-Wire Wire Line
-	8500 5800 8500 6000
-Wire Wire Line
-	9650 5800 9650 6000
-Wire Wire Line
-	9400 5400 9650 5400
-Wire Wire Line
-	9650 5400 9650 5600
-Wire Wire Line
-	8500 5600 8500 5400
-Wire Wire Line
-	8500 5400 8800 5400
+P 9950 5975
+F 0 "#PWR017" H 9950 5725 50  0001 C CNN
+F 1 "GND" H 9955 5802 50  0000 C CNN
+F 2 "" H 9950 5975 50  0001 C CNN
+F 3 "" H 9950 5975 50  0001 C CNN
+	1    9950 5975
+	1    0    0    -1
+$EndComp
+Wire Wire Line
+	9950 5775 9950 5975
+Wire Wire Line
+	9700 5375 9950 5375
+Wire Wire Line
+	9950 5375 9950 5575
+Wire Wire Line
+	8200 5375 8500 5375
 $Comp
 L archive:power_+3V3 #PWR018
 U 1 1 60DB2DA4
-P 9900 5250
-F 0 "#PWR018" H 9900 5100 50  0001 C CNN
-F 1 "+3V3" H 9915 5423 50  0000 C CNN
-F 2 "" H 9900 5250 50  0001 C CNN
-F 3 "" H 9900 5250 50  0001 C CNN
-	1    9900 5250
-	1    0    0    -1
-$EndComp
-Wire Wire Line
-	9650 5400 9900 5400
-Wire Wire Line
-	9900 5400 9900 5250
-Connection ~ 9650 5400
+P 10200 5225
+F 0 "#PWR018" H 10200 5075 50  0001 C CNN
+F 1 "+3V3" H 10215 5398 50  0000 C CNN
+F 2 "" H 10200 5225 50  0001 C CNN
+F 3 "" H 10200 5225 50  0001 C CNN
+	1    10200 5225
+	1    0    0    -1
+$EndComp
+Wire Wire Line
+	9950 5375 10200 5375
+Wire Wire Line
+	10200 5375 10200 5225
+Connection ~ 9950 5375
 $Comp
 L archive:Device_R_Small R?
@@
 L archive:power_+5V #PWR014
 U 1 1 60EF9622
-P 8500 5250
-F 0 "#PWR014" H 8500 5100 50  0001 C CNN
-F 1 "+5V" H 8515 5423 50  0000 C CNN
-F 2 "" H 8500 5250 50  0001 C CNN
-F 3 "" H 8500 5250 50  0001 C CNN
-	1    8500 5250
-	1    0    0    -1
-$EndComp
-Wire Wire Line
-	8500 5250 8500 5400
-Connection ~ 8500 5400
+P 8200 5225
+F 0 "#PWR014" H 8200 5075 50  0001 C CNN
+F 1 "+5V" H 8215 5398 50  0000 C CNN
+F 2 "" H 8200 5225 50  0001 C CNN
+F 3 "" H 8200 5225 50  0001 C CNN
+	1    8200 5225
+	1    0    0    -1
+$EndComp
+Wire Wire Line
+	8200 5225 8200 5375
 Wire Notes Line
 	500  4350 11200 4350
@@
 	7300 3825 7300 3475
 Wire Notes Line
-	6950 6500 6950 4350
+	6975 6500 6975 4350
 Wire Wire Line
 	7350 1675 7350 1775
@@
 NoConn ~ 7200 2775
 Text Notes 750  2450 0    50   ~ 0
-The P channel Mosfet in series with the batery works as a\nsimple reverse polarity protection circuit.\n\nIf the battery is reversed it will not conduct, hence not turning the\ncircuit on.\n\nI didin't use the zenner on the gate because the Mosfet's maximum\nVgs voltage is higher than what we will be applied by the battery.\n\nAlso, I didin't use a resistor on the gate because the mosfet is \nconstantly on, wich means ringing will not occur.\n\nWatch this to learn more:\nhttps://www.youtube.com/watch?v=IrB-FPcv1Dc
+The P channel Mosfet in series with the batery works as a\nsimple reverse polarity protection circuit.\n\nIf the battery is reversed it will not conduct, hence not turning the\ncircuit on.\n\nI didin't use the zenner on the gate because the Mosfet's maximum\nVgs voltage is higher than what will be applied by the battery.\n\nAlso, I didin't use a resistor on the gate because the mosfet is \nconstantly on, wich means ringing will not occur.\n\nWatch this to learn more:\nhttps://www.youtube.com/watch?v=IrB-FPcv1Dc
 Text Notes 750  3700 0    50   ~ 0
-The MAX17201 is an I2C single cell battery monitor. Be aware of \nthe differences of the MAX17211, wich uses the 1-Wire protocol.\n\nThis component will measure the battery volatge and with the\n0.01 ohm shunt it will also measure the current.\n\nAlso be aware of the MAX17205, wich is a multiple cell monitor.
+The MAX17201 is an I2C single cell battery monitor. Be aware of \nthe differences of the MAX17211, wich uses the 1-Wire protocol.\n\nThis component will measure the battery voltage and using a\n0.01 ohm shunt it will also measure the current.\n\nAlso be aware of the MAX17205, wich is a multiple cell monitor.
 Wire Wire Line
 	4650 1475 4650 1575
-$Comp
-L archive:MSS-102545-14A-V-SMT_MSS-102545-14A-V-SMT S6
-U 1 1 6196346E
-P 2125 6100
-F 0 "S6" V 1950 6150 50  0000 L CNN
-F 1 "MSS-102545-14A-V-SMT" H 1375 6400 50  0000 L CNN
-F 2 "SW_MSS-102545-14A-V-SMT" H 2125 6100 50  0001 L BNN
-F 3 "" H 2125 6100 50  0001 L BNN
-F 4 "Manufacturer Recommendations" H 2125 6100 50  0001 L BNN "STANDARD"
-F 5 "1.0" H 2125 6100 50  0001 L BNN "PARTREV"
-F 6 "CUI Devices" H 2125 6100 50  0001 L BNN "MANUFACTURER"
-F 7 "2.7 mm" H 2125 6100 50  0001 L BNN "MAXIMUM_PACKAGE_HEIGHT"
-	1    2125 6100
-	-1   0    0    1
-$EndComp
 Text HLabel 1000 5650 0    50   Input ~ 0
 Pack
@@
 EndData
 $EndBitmap
+$Comp
+L SamacSys_Parts:TC1264-3.3VDB IC4
+U 1 1 62272C03
+P 9100 5425
+F 0 "IC4" H 9450 5625 50  0000 C CNN
+F 1 "TC1264-3.3VDB" H 9000 5625 50  0000 C CNN
+F 2 "SamacSys_Parts:SOT230P700X180-4N" H 10150 5525 50  0001 L CNN
+F 3 "http://ww1.microchip.com/downloads/en/devicedoc/21375d.pdf" H 10150 5425 50  0001 L CNN
+F 4 "LDO Regulator Pos 3.3V 0.8A Automotive 4-Pin(3+Tab) SOT-223 Tube" H 10150 5325 50  0001 L CNN "Description"
+F 5 "1.8" H 10150 5225 50  0001 L CNN "Height"
+F 6 "579-TC1264-3.3VDB" H 10150 5125 50  0001 L CNN "Mouser Part Number"
+F 7 "https://www.mouser.co.uk/ProductDetail/Microchip-Technology/TC1264-33VDB?qs=AkCjCAp%252BzjQSxS5e2ugTcA%3D%3D" H 10150 5025 50  0001 L CNN "Mouser Price/Stock"
+F 8 "Microchip" H 10150 4925 50  0001 L CNN "Manufacturer_Name"
+F 9 "TC1264-3.3VDB" H 10150 4825 50  0001 L CNN "Manufacturer_Part_Number"
+	1    9100 5425
+	1    0    0    -1
+$EndComp
+Wire Wire Line
+	9050 5875 9050 5950
+Wire Wire Line
+	9050 5950 9100 5950
+Wire Wire Line
+	9150 5950 9150 5875
+Wire Wire Line
+	9100 6000 9100 5950
+Connection ~ 9100 5950
+Wire Wire Line
+	9100 5950 9150 5950
+$Comp
+L archive:MSS-102545-14A-V-SMT_MSS-102545-14A-V-SMT S6
+U 1 1 6196346E
+P 2125 6100
+F 0 "S6" V 1950 6150 50  0000 L CNN
+F 1 "MSS-102545-14A-V-SMT" H 1375 6400 50  0000 L CNN
+F 2 "SW_MSS-102545-14A-V-SMT" H 2125 6100 50  0001 L BNN
+F 3 "" H 2125 6100 50  0001 L BNN
+F 4 "Manufacturer Recommendations" H 2125 6100 50  0001 L BNN "STANDARD"
+F 5 "1.0" H 2125 6100 50  0001 L BNN "PARTREV"
+F 6 "CUI Devices" H 2125 6100 50  0001 L BNN "MANUFACTURER"
+F 7 "2.7 mm" H 2125 6100 50  0001 L BNN "MAXIMUM_PACKAGE_HEIGHT"
+	1    2125 6100
+	-1   0    0    -1
+$EndComp
+Text Notes 8625 5700 2    50   ~ 0
+There's no capacitor in the input\nbecause C10 and C8 are placed\nnear the regulator on the PCB.
 $EndSCHEMATC

Commit message: Reduces board length to 101,5 mm
JLC PCB allows a 4 layer PCB to be manufactured for just $8,00 if it is within 102 x 102 mm. The previous version was 105,47 mm, making it cost $37,00.

To reduce the manufacturing cost the board had its size cut down to 101,5 mm. This was possible by moving the buzzer from the top left corner of the board to the free space between the two SMA connectors.
Parts:
- IC4: symbol SamacSys_Parts:TC1264-3.3VDB -> archive:SamacSys_Parts_TC1264-3.3VDB
Changed lines of the file:
@@
 $EndBitmap
 $Comp
-L SamacSys_Parts:TC1264-3.3VDB IC4
+L archive:SamacSys_Parts_TC1264-3.3VDB IC4
 U 1 1 62272C03
 P 9100 5425
